File: Synthtar/indicator_assembly.sch (EAGLE design)
At the start: 82 parts, among them IC1 74HC164N, IC2 4081N, IC3 555, IC4 4081N, J1 AUDIO_JACK_3.5MM_PTH, M1 ARDUINO-NANO-3.0, X1 HD44780LCD-1602, X2 MINI-USB-UX60A-MB-5ST

Commit message: Board building
started migrating overall schematic into individual boards
Parts:
- removed D1, D10, D11, D12, D13, D14, D15, D16, D17, D18, D2, D3, D4, D5, D6, D7, D8, D9: 200mA/100V/1V, SparkFun-DiscreteSemi:DIODE-1N4148
- removed IC4: 4081N, 40xx:4081N
- removed J1: AUDIO_JACK_3.5MM_PTH, SparkFun-Connectors:AUDIO_JACK_3.5MM_PTH
- removed M1: ARDUINO-NANO-3.0, diy-modules:ARDUINO-NANO-3.0
- removed R1, R20, R4: 220, rcl:R-US_0204/7
- removed R10, R11, R12, R13: 10k, rcl:R-US_0204/7
- removed R14, R16, R18, R2, R3: 10k, pot:TRIM_US-B64Y
- removed R17, R19: 4.7k, rcl:R-US_0204/7
- removed S1, S10, S11, S12, S13, S14, S15, S16, S18, S19, S2, S3, S4, S5, S6, S7, S8, S9: (no value), switch-omron:10-XX
- removed S17: (no value), SparkFun-Switches:SWITCH-DPDT-PTH-GPI-152-3013
- removed SP1, SP2: SMS-1308MS-2-R, speaker:SMS-1308MS-2-R
- removed U$1: MIDIJACK, adafruit:MIDIJACK
- removed U$2: AUDIO_AMP, synthtar:AUDIO_AMP
- removed U$3: CHARGER, synthtar:CHARGER
- removed U$4: VBOOST, synthtar:VBOOST
- removed U$5: TEENSY_LC_ALL_PINS, Teensy_3_and_LC_Series_Boards_v1.4:TEENSY_LC_ALL_PINS
- removed U$6: LEVEL-SHIFTER-4CH, diy-modules:LEVEL-SHIFTER-4CH
- removed VS1: VS1053B, synthtar:VS1053B
- removed X1: HD44780LCD-1602, adafruit:HD44780LCD-1602
- removed X2: MINI-USB-UX60A-MB-5ST, con-hirose:MINI-USB-UX60A-MB-5ST
Connections:
- removed net ADD_BTNS: S18.P, S19.P, U$5.6/PWM
- removed net A_IN2: R14.S, U$5.15/A1/T
- removed net A_IN3: R16.S, U$5.16/A2/PWM/T
- removed net A_IN4: R18.S, U$5.17/A3/PWM/T
- removed net BODY_BTNS: S1.P1, S2.P1, S3.P1, S4.P1, U$5.3/T/PWM
- removed net B_ROW_1: D1.C, D13.C, D17.C, D5.C, D9.C, R10.1, U$5.9/RX2/PWM
- removed net B_ROW_2: D10.C, D14.C, D18.C, D2.C, D6.C, R11.1, U$5.10/TX2/PWM
- removed net B_ROW_3: D11.C, D15.C, D3.C, D7.C, R12.1, U$5.11/MOSI
- removed net B_ROW_4: D12.C, D16.C, D4.C, D8.C, R13.1, U$5.12/MISO
- removed net MENU_BTNS: S10.P, S11.P, S12.P, S9.P, U$5.4/T/PWM
- removed net N$1: M1.D4, X1.RS
- removed net N$10: R17.1, U$5.22/A8/T/PWM/SCL1
- removed net N$11: R20.2
- removed net N$12: U$3.LOAD+, U$4.VIN+
- removed net N$13: D1.A, S5.S
- removed net N$15: U$3.LOAD-, U$4.VIN-
- removed net N$16: M1.D5, X1.E
- removed net N$18: U$2.GAIN3
- removed net N$19: M1.D6, X1.DB4
- removed net N$2: X2.2
- removed net N$20: D2.A, S6.S
- removed net N$21: D3.A, S7.S
- removed net N$22: VS1.1, VS1.3V3
- removed net N$23: D4.A, S8.S
- removed net N$24: D5.A, S9.S
- removed net N$25: J1.TIP, U$2.L+, VS1.LOUT
- removed net N$26: J1.SLEEVE, U$2.R+, VS1.ROUT
- removed net N$27: SP2.1, U$2.ROUT+
- removed net N$28: SP2.2, U$2.ROUT-
- removed net N$29: SP1.2, U$2.LOUT+
- removed net N$3: X2.3
- removed net N$30: SP1.1, U$2.LOUT-
- removed net N$31: D6.A, S10.S
- removed net N$32: J1.RSH, U$2.L-, U$2.R-, VS1.AGND1
- removed net N$33: D7.A, S11.S
- removed net N$34: D8.A, S12.S
- removed net N$35: D9.A, S1.S
- removed net N$36: U$2.GAIN4
- removed net N$37: D10.A, S2.S
- removed net N$38: D11.A, S3.S
- removed net N$39: D12.A, S4.S
- removed net N$4: U$3.DCIN+, X2.1
- removed net N$40: U$2.GAIN7, U$2.GAIN8
- removed net N$41: D13.A, S13.S
- removed net N$42: D14.A, S14.S
- removed net N$43: D15.A, S15.S
- removed net N$44: D16.A, S16.S
- removed net N$45: R4.2, U$1G$1.4
- removed net N$46: R20.1, U$1G$1.5
- removed net N$48: M1.D7, X1.DB5
- removed net N$5: U$3.DCIN-, X2.5
- removed net N$52: M1.D8, X1.DB6
- removed net N$53: M1.D9, X1.DB7
- removed net N$6: D17.A, S18.S
- removed net N$63: R1.2, X1.A
- removed net N$64: R3.S, X1.VO
- removed net N$7: D18.A, S19.S
- removed net N$8: R19.1, U$5.23/A9/T/PWM/SDA1
- removed net N$9: S17.5
- removed net NECK_BTNS: S5.P, S6.P, S7.P, S8.P, U$5.2
- removed net QUIK_BTNS: S13.P, S14.P, S15.P, S16.P, U$5.5
- removed net SCREEN_BUSYHV: M1.D2, U$6.HV4
- removed net SCREEN_BUSYLV: U$6.LV4
- removed net SCREEN_DATAHV: M1.D0/RX, U$6.HV1
- removed net SCREEN_DATALV: U$5.1/TX1/T/MISO1, U$6.LV1
- removed net VCC: R14.A, R16.A, R17.2, R18.A, R19.2, R2.A, U$5.3.3V, U$6.LV
- removed net VOL_RD: R2.S, U$5.14/A0
- removed net VS_MIDI: IC4A.I0, IC4A.I1, U$5.8/TX3, VS1.RX
- removed net VS_RST: U$5.20/A6/PWM/SCK1, VS1.RST
- net +5V: no longer IC4P.VDD, M1.5V, R1.1, R3.E, R4.1, U$2.VDD, U$4.VOUT+, U$5.VIN, VS1.VCC, X1.VDD
- net AMP_SDWN: no longer S17.2, U$2.SDWN
- net GND: no longer IC4P.VSS, M1.GND.2, R10.2, R11.2, R12.2, R13.2, R14.E, R16.E, R18.E, R2.E, R3.A, S17.3, U$1G$1.2, U$2.GND, U$4.VOUT-, U$5.GND, U$6.GND.1, VS1.0, VS1.GND, X1.K, X1.RW, X1.VSS
- net SR_CLK: no longer U$5.19/A5/T/SCL
- net SR_DATA: no longer U$5.18/A4/T/SDA
Other:
- note removed: "10ks here because 100k makes RC time constant with pin too high"
- note removed: "3.3v/10k=.33mA"
- note removed: "ADD DECOUPLING CAPS"
- note removed: "BATTERY HERE"
- note removed: "BLAKE NEMETH"
- note removed: "BODY BUTTONS AND SWITCHES"
- note removed: "CHARGE HERE"
- note removed: "Draws ~2mA while active and not playing sound. Playing sound at average volume (40) draws an additional 3mA."
- note removed: "It = .33mA * 4 = 1.32mA"
- note removed: "MENU BUTTONS"
- note removed: "NECK BUTTONS"
- note removed: "P = 3.3^2/10000 = 1.089mW"
- note removed: "POWER SUPPLY"
- note removed: "Pt(Analog) = 1.089mW * 4 = 4.356mW"
- note removed: "Use a shift register to control indicators?"
- note removed: "amp on"
- note removed: "backlight power"
- note removed: "contrast adjust"
- note removed: "d+"
- note removed: "d-"
- note removed: "if you plug in headphones while amp is playing it can shock the vs1053b"
- note removed: "may need a distribution amp here to isolate"
- note removed: "midi out"
- note removed: "need to measure this current"
- note removed: "or having both!"
- note removed: "other analog controls"
- note removed: "over 3.3v on the digital pins can fry teensy lc..."
- note removed: "quick buttonas"
- note removed: "reserved for i2c"
- note removed: "rethinking these, may do mechanical switch because i don't like how the latching switches feel"
- note removed: "sdown pulled to ground shuts off amp, floating turns it on"
- note removed: "thinking about replacing this midi jack with usb midi functionality"
- note removed: "voume control"
- moved on the sheet: C1, C2, C3, D19, IC1, IC1P, IC2A, IC2B, IC2C, IC2D, IC2P, IC3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
