File: Synthtar/indicator_assembly.sch (EAGLE design)
At the start: 23 parts, among them IC1 74HC164N, IC2 4081N, IC3 555

Commit message: indicator update
honestly don't remmember what i changed, looks like added a header maybe?
Other:
- note added: "blue"
- note added: "green"
- note added: "red"
Changed lines of the file:
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@@
 <text x="190.5" y="73.66" size="1.778" layer="91">for mounting the leds on the case at various locations</text>
 <text x="193.04" y="38.1" size="1.778" layer="91">redo these resistor calcs based on color</text>
+<text x="208.28" y="66.04" size="1.778" layer="91">green</text>
+<text x="208.28" y="12.7" size="1.778" layer="91">blue</text>
+<text x="208.28" y="27.94" size="1.778" layer="91">red</text>
+<text x="208.28" y="48.26" size="1.778" layer="91">red</text>
 </plain>
 <instances>
