File: Synthtar/neck_assembly.sch (EAGLE design)
At the start: 9 parts

Commit message: misc changes
misc updates while doing documentation
Other:
- note added: "headers, the switches will be mounted externally"
- note removed: "replace these with headers, the switches will be mounted externally"
Changed lines of the file:
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@@
 <wire x1="100.33" y1="74.93" x2="36.83" y2="74.93" width="0.1524" layer="97"/>
 <text x="80.01" y="72.39" size="1.778" layer="97">NECK BUTTONS</text>
-<text x="92.71" y="59.69" size="1.778" layer="91">replace these with headers, the switches will be mounted externally</text>
-<text x="92.71" y="57.15" size="1.778" layer="91">2 pin headers</text>
+<text x="97.79" y="59.69" size="1.778" layer="91">headers, the switches will be mounted externally</text>
+<text x="97.79" y="57.15" size="1.778" layer="91">2 pin headers</text>
 <text x="92.71" y="45.72" size="1.778" layer="91">diodes on board so switches have no polarity</text>
 <text x="2.54" y="50.8" size="1.778" layer="91">ribbon cable? maybe</text>
