File: Synthtar/overall_schem.sch (EAGLE design)
At the start: 83 parts, among them IC2 4081N, IC3 555, IC4 4081N, J1 AUDIO_JACK_3.5MM_PTH, M1 ARDUINO-NANO-3.0, U1 JOYSTICKPTH, X1 HD44780LCD-1602, X2 MINI-USB-UX60A-MB-5ST

Commit message: so fucking much
a
Parts:
- removed C1: .47uF, rcl:CPOL-USE2-4
- removed C2: .01uF, rcl:C-US025-030X050
- removed D19: 200mA/100V/1V, SparkFun-DiscreteSemi:DIODE-1N4148
- removed IC3: 555, SparkFun-IC-Special-Function:555P
- removed R15: 2k, rcl:R-US_0204/7
- removed R17, R19: 4.7k, rcl:R-US_0204/7
- removed R9: 1k, rcl:R-US_0204/7
- added C4: .1uF, rcl:C-US025-024X044
- added U$13: LCD-I2C-CONVERTER, diy-modules:LCD-I2C-CONVERTER
- C3: value .1uF -> .01uF; device rcl:C-US025-030X050 -> rcl:C-US025-024X044
- R5: value 400 -> 580
- R6, R7: value 400 -> 600
- R8: value 400 -> 620
Connections:
- removed net SR_CLK: U$5.19/A5/T/SCL
- new net +5V1: C3.1, C4.1
- new net A_ACTIVE: R14.A, R16.A, R18.A, R2.A, U$5.19/A5/T/SCL, U1.V+
- new net GND1: C3.2, C4.2
- new net N$10: M1.A4, U$13.SDA
- new net N$66: U$13.DB0, X1.DB0
- new net N$71: U$13.EN, X1.E
- new net N$72: U$13.RS, X1.RS
- new net N$73: U$13.R/W, X1.RW
- new net N$74: M1.D8
- new net N$75: M1.D9
- new net VDD: U$13.VDD, X1.VDD
- new net VSS: U$13.VSS, X1.VSS
- net +5V: no longer R1.1, X1.VDD
- net GND: no longer C1.-, C2.2, C3.2, IC3.GND, X1.K, X1.RW, X1.VSS
- net I2C_SCL: no longer R17.1
- net I2C_SDA: no longer R19.1
- net IND_PWM: now also M1.D5; no longer IC3.OUT
- net N$1: now also R3.S, U$13.VEE, X1.VO; no longer M1.D4, X1.RS
- net N$11: now also IC4A.O
- net N$16: now also U$13.LED.K, X1.K; no longer M1.D5, X1.E
- net N$19: now also M1.A5, U$13.SCL; no longer M1.D6, X1.DB4
- net N$48: now also R1.1, U$13.LED.A; no longer M1.D7, X1.DB5
- net N$52: now also U$13.DB7, X1.DB7; no longer M1.D8, X1.DB6
- net N$53: now also U$13.DB6, X1.DB6; no longer M1.D9, X1.DB7
- net N$59: now also U$13.DB5, X1.DB5; no longer IC3.TRE, IC3.TRI
- net N$60: now also U$13.DB4, X1.DB4; no longer D19.A, IC3.DIS, R15.1, R9.2
- net N$61: now also U$13.DB3, X1.DB3; no longer C2.1, IC3.CON
- net N$62: now also U$13.DB2, X1.DB2; no longer C1.+, D19.C, R15.2
- net N$64: now also M1.D7; no longer R3.S, X1.VO
- net N$65: now also U$13.DB1, X1.DB1; no longer C3.1, IC3./RES, IC3.VCC+, R9.1
- net VCC: no longer R14.A, R16.A, R17.2, R18.A, R19.2, R2.A, U1.V+
Other:
- note added: ".26mA/100 = 2.6uA"
- note added: ".5mA leakage when amp off - 5*.5mA = 2.5mW"
- note added: "18 buttons: 8.58uW*18 = 154.44uW"
- note added: "2.9/5mA = 580"
- note added: "2mA*5v=10mW (idle)"
- note added: "3.1/5mA=620"
- note added: "3/5mA = 600"
- note added: "5.445mW/100 = 54.45uW"
- note added: "5mA*5v=25mW (playing)"
- note added: "5v*18mA = 90mW"
- note added: "5v*20mA=100mW"
- note added: "5v-2v/220=i=13.6mA p=vi=5*13.6mA=68.18mW"
- note added: "5v^2/10k=2.5mW"
- note added: "It = .33mA * 5 = 1.65mA"
- note added: "Pt(Analog) = 1.089mW * 5 = 5.445mW"
- note added: "active <1% of the time, assume 1% for calcs"
- note added: "active approx 1% of the time"
- note added: "amp - blue"
- note added: "current: 3.3-.7/10000 = .26mA (when active)"
- note added: "d7"
- note added: "d8"
- note added: "d9"
- note added: "idle draw about 20mA because I haven't modded my nano yet"
- note added: "m2 - red"
- note added: "m4 -red"
- note added: "negligible current, uses FETs"
- note added: "not used in prototype"
- note added: "p=vi -> i = p/v 390.21mW/5v = 78mA"
- note added: "pow = 2.6uA * 3.3v = 8.58uW (per button)"
- note added: "power - green"
- note added: "prototype has usb midi"
- note added: "screen + indicators"
- note added: "total power: +90mW (teensy) +100mW (nano) +100mW (vs1053b) +70mW (screen) +54.45uW (analog) +154.44uW (matrix) +30mW (indicators) -------------------------- 390.21mW"
- note added: "vf = 2.9v"
- note added: "vf = 2v"
- note added: "vf = 3.1v"
- note added: "vr = 2.9v"
- note added: "vr = 3.1v"
- note added: "vr = 3v"
- note added: "~10-15mA draw, assume 18mA max"
- note added: "~20mA for all of this, never did individual measurements on each component 5v*20mA=100mW"
- note removed: "It = .33mA * 4 = 1.32mA"
- note removed: "Pt(Analog) = 1.089mW * 4 = 4.356mW"
- note removed: "Use a shift register to control indicators?"
- note removed: "allows for toggling PWM'd led's with dc voltages with no cpu overhead"
- note removed: "idle current to run this is about 1.5mA. Could reduce, but would require bigger capacitor"
- note removed: "or having both!"
- note removed: "power draw: 5v*1.5mA=7.5mW"
- note removed: "rethinking these, may do mechanical switch because i don't like how the latching switches feel"
- note removed: "this circuit generates a 30% duty cycle PWM signal at 1kHz"
- note removed: "this circuit uses CMOS AND gates to control LEDs with a PWM input (so they can all be dimmed)"
- moved on the sheet: C3, IC2A, IC2B, IC2C, IC2D, IC2P, IC4A, IC4P, LED3, LED4, LED5, LED6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

Commit message: added code for screenslave and main teensy
also fixed some resistor values in overall schem
Parts:
- R5: value 580 -> 380
- R8: value 620 -> 420
Other:
- note added: "1.9/5mA = 380"
- note added: "2.1/5mA=420"
- note added: "vr = 1.9v"
- note added: "vr = 2.1v"
- note removed: "2.9/5mA = 580"
- note removed: "3.1/5mA=620"
- note removed: "vr = 2.9v"
- note removed: "vr = 3.1v"
Changed lines of the file:
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@@
 <part name="IC2" library="40xx" library_urn="urn:adsk.eagle:library:80" deviceset="4081" device="N" package3d_urn="urn:adsk.eagle:package:820/2"/>
 <part name="LED3" library="led" library_urn="urn:adsk.eagle:library:259" deviceset="LED" device="5MM" package3d_urn="urn:adsk.eagle:package:15799/2"/>
-<part name="R5" library="rcl" library_urn="urn:adsk.eagle:library:334" deviceset="R-US_" device="0204/7" package3d_urn="urn:adsk.eagle:package:23498/1" value="580"/>
+<part name="R5" library="rcl" library_urn="urn:adsk.eagle:library:334" deviceset="R-US_" device="0204/7" package3d_urn="urn:adsk.eagle:package:23498/1" value="380"/>
 <part name="SUPPLY14" library="supply2" library_urn="urn:adsk.eagle:library:372" deviceset="GND" device=""/>
 <part name="LED4" library="led" library_urn="urn:adsk.eagle:library:259" deviceset="LED" device="5MM" package3d_urn="urn:adsk.eagle:package:15799/2"/>
@@
 <part name="SUPPLY20" library="supply2" library_urn="urn:adsk.eagle:library:372" deviceset="GND" device=""/>
 <part name="LED6" library="led" library_urn="urn:adsk.eagle:library:259" deviceset="LED" device="5MM" package3d_urn="urn:adsk.eagle:package:15799/2"/>
-<part name="R8" library="rcl" library_urn="urn:adsk.eagle:library:334" deviceset="R-US_" device="0204/7" package3d_urn="urn:adsk.eagle:package:23498/1" value="620"/>
+<part name="R8" library="rcl" library_urn="urn:adsk.eagle:library:334" deviceset="R-US_" device="0204/7" package3d_urn="urn:adsk.eagle:package:23498/1" value="420"/>
 <part name="SUPPLY30" library="supply2" library_urn="urn:adsk.eagle:library:372" deviceset="GND" device=""/>
 <part name="IC4" library="40xx" library_urn="urn:adsk.eagle:library:80" deviceset="4081" device="N" package3d_urn="urn:adsk.eagle:package:820/2"/>
@@
 <text x="264.16" y="22.86" size="1.778" layer="97">vf = 2v</text>
 <text x="271.78" y="10.16" size="1.778" layer="97">vf = 2.9v</text>
-<text x="271.78" y="55.88" size="1.778" layer="97">vr = 2.9v</text>
-<text x="271.78" y="7.62" size="1.778" layer="97">vr = 3.1v</text>
+<text x="271.78" y="55.88" size="1.778" layer="97">vr = 1.9v</text>
+<text x="271.78" y="7.62" size="1.778" layer="97">vr = 2.1v</text>
 <text x="269.24" y="43.18" size="1.778" layer="97">vr = 3v</text>
 <text x="264.16" y="20.32" size="1.778" layer="97">vr = 3v</text>
-<text x="284.48" y="55.88" size="1.778" layer="97">2.9/5mA = 580</text>
+<text x="284.48" y="55.88" size="1.778" layer="97">1.9/5mA = 380</text>
 <text x="279.4" y="43.18" size="1.778" layer="97">3/5mA = 600</text>
 <text x="274.32" y="20.32" size="1.778" layer="97">3/5mA = 600</text>
-<text x="284.48" y="7.62" size="1.778" layer="97">3.1/5mA=620</text>
+<text x="284.48" y="7.62" size="1.778" layer="97">2.1/5mA=420</text>
 <text x="-86.36" y="-20.32" size="1.778" layer="97">screen + indicators</text>
 <text x="66.04" y="-27.94" size="1.778" layer="97">5v^2/10k=2.5mW</text>
